File: HPM5E31.kicad_pcb (KiCad board)
At the start: 4 copper layers, 75 x 50 mm, 202 parts, among them J1 Conn_ARM_JTAG_SWD_10, J10 Conn_01x06_MountingPin, J11 Conn_01x03_Pin, J12 Conn_01x04_MountingPin, J13 Conn_01x06_MountingPin, J14 USB_C_Receptacle_USB2.0_16P, J15 Conn_01x03_Socket, J16 Conn_01x04_Socket, J2 Conn_01x03_MountingPin, J3 RJ45_Hanrun_HR911105A_Horizon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, J4 Conn_01x04_MountingPin, J5 Conn_01x03_Pin, J6 Conn_01x02_MountingPin, J7 Conn_01x06_MountingPin, J8 Conn_01x06_MountingPin, J9 Conn_01x06_MountingPin, Q1 SS8050, Q2 SS8050, SW1 SW_Push, U1 HPM5E31IPB1, U10 REF3033, U11 RY8411, U12 XC6210B332MR, U13 AFA11-S08GLA-00, U2 LAN8720A, U4 MLT-5020, U5 TJA1051TK-3, U6 RTL8211F-CG, U7 7*7*5-6P-L WX, U8 HR911130A, U9 USBLC6-2SC6, Y1 24Mhz, Y2 X322525MOB4SI, Y3 X322525MOB4SI

Commit message: Update KiCad project files
Parts:
- removed C16: 100nF, Capacitor_SMD:C_0603_1608Metric
- removed FL1: Filter_EMI_LL_1423, Inductor_SMD:L_CommonModeChoke_Coilank_ACM2012
- removed J1: Conn_ARM_JTAG_SWD_10, Connector_PinHeader_1.27mm:PinHeader_2x05_P1.27mm_Vertical
- added R69: 0R, Resistor_SMD:R_0603_1608Metric, F.Cu at (228.1, 67.6)
- added U3: HX JN1.27-2X6P ZZ H4.9, mylib:HX_JN1_27-2X6P_ZZ_H4_9_C42372548, F.Cu at (208.1, 100.0)
- moved D1 30.1 mm to (207.4, 67.7), turned to -90 degrees
- moved R7 29.2 mm to (208.9, 67.7), turned to -90 degrees
- moved Q2 4.93 mm to (192.5, 94.3)
- moved R21 4.93 mm to (190.1, 94.2)
- moved R20 4.93 mm to (194.6, 94.3)
- moved D5 1.58 mm to (234.4, 73.7)
- moved D7 1.58 mm to (234.4, 80.5)
- moved D6 1.58 mm to (234.4, 77.1)
- moved D8 1.58 mm to (234.4, 84.1)
- moved D12 0.84 mm to (210.3, 67.7)
- moved R14 0.81 mm to (211.7, 67.7)
- moved D13 0.78 mm to (213.1, 67.7)
- moved R15 0.75 mm to (214.5, 67.7)
- moved D14 0.72 mm to (215.9, 67.7)
- moved R68 0.68 mm to (217.4, 67.7)
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Connections:
- U1 pad 24: /PIN_A/ESC_RST -> /PIN_A/ESC0.REFCK
- U1 pad 5: /PIN_A/ESC0.REFCK -> /PIN_A/ESC_RST
- U9 pad 4: Net-(FL1-Pad2) -> /Crystal/USB_DP
- U9 pad 6: Net-(FL1-Pad1) -> /Crystal/USB_DN
Routing:
- net /PIN_A/LED: track 3.95 -> 34.6 mm
- net /PIN_A/UART0.TXD: track 24.8 -> 33.6 mm
- net /PIN_F/ETH0.RXD1: track 19.9 -> 27.2 mm
- net /PIN_A/ESC_RST: track 23.6 -> 30.4 mm, vias 2 -> 0
- net /PIN_F/ETH0.RXDV: track 18.9 -> 25.4 mm
- net /PIN_A/ESC0.REFCK: track 29.3 -> 23.9 mm, vias 0 -> 2
- net /Crystal/USB_DP: track 58.4 -> 62.8 mm
- net Net-(J11-Pin_1): track 10.2 -> 5.85 mm
- net /PIN_BCD/DC: track 22.3 -> 18.0 mm
- net GND: track 125.8 -> 129.9 mm, vias 320 -> 294
- net /PIN_BCD/SPI1.CS0: track 19.8 -> 23.7 mm, vias 0 -> 2
- net /Crystal/USB_DN: track 58.0 -> 61.8 mm
- net /PIN_A/UART0.RXD: track 20.4 -> 23.9 mm
- net /PIN_F/MDIP3: track 18.1 -> 14.9 mm
- net /PIN_BCD/SPI1.MOSI: track 25.4 -> 22.2 mm
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Other:
- board text added: "HPM5E31_V0.3"
- board text removed: "HPM5E31_V0.2"
