File: PIN_A.kicad_sch (KiCad schematic)
At the start: 52 parts, among them J1 Conn_ARM_JTAG_SWD_10, J15 Conn_01x03_Socket, J2 Conn_01x03_MountingPin, J3 RJ45_Hanrun_HR911105A_Horizon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, Q1 SS8050, U1 HPM5E31IPB1, U2 LAN8720A, U4 MLT-5020, Y2 X322525MOB4SI

Commit message: Update KiCad project files
Parts:
- removed C16: 100nF, Capacitor_SMD:C_0603_1608Metric, symbol Device:C
- removed J1: Conn_ARM_JTAG_SWD_10, Connector_PinHeader_1.27mm:PinHeader_2x05_P1.27mm_Vertical, symbol Connector:Conn_ARM_JTAG_SWD_10
- added U3: HX JN1.27-2X6P ZZ H4.9, mylib:HX_JN1_27-2X6P_ZZ_H4_9_C42372548, symbol mylib:HX_JN1_27-2X6P_ZZ_H4_9_C42372548
Connections:
- net +3.3V: now also U3.1
- net ESC0.REFCK: now also U1.24 (PA24/GPTMR2.COMP1/UART6.TXD/SPI3.CS2/ESC0.P0_TXCK); no longer U1.5 (PA09/GPTMR0.CAPT1/UART2.RXD/I2C0.SDA/MCAN2.RXD/ESC0.REFCK/PWM1.P1/TRGM.P09)
- net ESC_RST: now also U1.5 (PA09/GPTMR0.CAPT1/UART2.RXD/I2C0.SDA/MCAN2.RXD/ESC0.REFCK/PWM1.P1/TRGM.P09); no longer U1.24 (PA24/GPTMR2.COMP1/UART6.TXD/SPI3.CS2/ESC0.P0_TXCK)
- net GND: now also U3.3, U3.5, U3.7, U3.9
- net JTAG.TCK: now also U3.4
- net JTAG.TDI: now also U3.8
- net JTAG.TDO: now also U3.6
- net JTAG.TMS: now also U3.2
- net JTAG.TRST: now also U3.10
- net UART0.RXD: now also U3.12
- net UART0.TXD: now also U3.11
