File: PIN_F.kicad_sch (KiCad schematic)
At the start: 76 parts, among them J13 Conn_01x06_MountingPin, U1 HPM5E31IPB1, U6 RTL8211F-CG, U7 7*7*5-6P-L WX, U8 HR911130A, Y3 X322525MOB4SI

Commit message: Update KiCad project files
Parts:
- added R69: 0R, Resistor_SMD:R_0603_1608Metric, symbol Device:R
Connections:
- net VCC3V3_PHY: now also R69.2
- net VCCIO_PHY: now also R69.1
Changed lines of the file:
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@@
 	(wire
 		(pts
+			(xy 156.21 229.87) (xy 163.83 229.87)
+		)
+		(stroke
+			(width 0)
+			(type default)
+		)
+	)
+	(wire
+		(pts
 			(xy 181.61 143.51) (xy 190.5 143.51)
 		)
@@
 	(wire
 		(pts
+			(xy 144.78 223.52) (xy 144.78 229.87)
+		)
+		(stroke
+			(width 0)
+			(type default)
+		)
+	)
+	(wire
+		(pts
 			(xy 236.22 140.97) (xy 254 140.97)
 		)
@@
 	(wire
 		(pts
+			(xy 163.83 229.87) (xy 163.83 223.52)
+		)
+		(stroke
+			(width 0)
+			(type default)
+		)
+	)
+	(wire
+		(pts
 			(xy 335.28 50.8) (xy 344.17 50.8)
 		)
@@
 	(wire
 		(pts
+			(xy 144.78 229.87) (xy 148.59 229.87)
+		)
+		(stroke
+			(width 0)
+			(type default)
+		)
+	)
+	(wire
+		(pts
 			(xy 265.43 207.01) (xy 273.05 207.01)
 		)
@@
 		)
 	)
+	(label "VCCIO_PHY"
+		(at 144.78 223.52 180)
+		(effects
+			(font
+				(size 1.27 1.27)
+			)
+			(justify right bottom)
+		)
+	)
 	(label "MDIP3"
 		(at 317.5 115.57 0)
@@
 	)
 	(label "VCC3V3_PHY"
+		(at 163.83 223.52 180)
+		(effects
+			(font
+				(size 1.27 1.27)
+			)
+			(justify right bottom)
+		)
+	)
+	(label "VCC3V3_PHY"
 		(at 144.78 195.58 180)
 		(effects
@@
 					(unit 1)
 				)
+			)
+		)
+	)
+	(symbol
+		(lib_id "Device:R")
+		(at 152.4 229.87 90)
+		(unit 1)
+		(body_style 1)
+		(exclude_from_sim no)
+		(in_bom yes)
+		(on_board yes)
+		(in_pos_files yes)
+		(dnp no)
+		(property "Reference" "R69"
+			(at 147.32 227.33 0)
+			(show_name no)
+			(do_not_autoplace no)
+			(effects
+				(font
+					(size 1.27 1.27)
+				)
+			)
+		)
+		(property "Value" "0R"
+			(at 157.48 227.33 0)
+			(show_name no)
+			(do_not_autoplace no)
+			(effects
+				(font
+					(size 1.27 1.27)
+				)
+			)
+		)
+		(property "Footprint" "Resistor_SMD:R_0603_1608Metric"
+			(at 152.4 231.648 90)
+			(hide yes)
+			(show_name no)
+			(do_not_autoplace no)
+			(effects
+				(font
+					(size 1.27 1.27)
+				)
+			)
+		)
+		(property "Datasheet" ""
+			(at 152.4 229.87 0)
+			(hide yes)
+			(show_name no)
+			(do_not_autoplace no)
+			(effects
+				(font
+					(size 1.27 1.27)
+				)
+			)
+		)
+		(property "Description" "Resistor"
+			(at 152.4 229.87 0)
+			(hide yes)
+			(show_name no)
+			(do_not_autoplace no)
+			(effects
+				(font
+					(size 1.27 1.27)
+				)
+			)
+		)
+		(property "KLC_S3.3" ""
+			(at 152.4 229.87 0)
+			(hide yes)
+			(show_name no)
+			(do_not_autoplace no)
+			(effects
+				(font
+					(size 1.27 1.27)
+				)
+			)
+		)
+		(property "KLC_S4.1" ""
+			(at 152.4 229.87 0)
+			(hide yes)
+			(show_name no)
+			(do_not_autoplace no)
+			(effects
+				(font
+					(size 1.27 1.27)
+				)
+			)
+		)
+		(pin "2"
+		)
+		(pin "1"
+		)
+		(instances
+			(project "HPM5E31"
+				(path "/c97d420a-5bfd-40ab-9a74-5349ba6434d5/66409916-63cc-4ec6-a4ee-7afe73c5271b"
+					(reference "R69")
+					(unit 1)
+				)
